File: Control Keys.sch (KiCad schematic (older format))
At the start: 0 parts

Commit message: Schematic completed first draft
Parts:
- added C? (x2): 1n, symbol Device:C
- added U? (x2): 74LS597, symbol 74xx_IEEE:74LS597
Connections:
- new net: U?.14 (SER), U?.9 (QH)
- new net DEL: U?.6 (G)
- new net DN: U?.3 (D)
- new net END: U?.7 (H)
- new net EXT10: U?.7 (H)
- new net EXT8: U?.5 (F)
- new net EXT9: U?.6 (G)
- new net GND: C?.2, C?.2, U?.13 (~SLoad), U?.13 (~SLoad), U?.14 (SER), U?.8 (GND), U?.8 (GND)
- new net HOME: U?.4 (E)
- new net INS: U?.3 (D)
- new net LT: U?.2 (C)
- new net PAUS: U?.2 (C)
- new net PGDN: U?.15 (A)
- new net PGUP: U?.5 (F)
- new net PRNT: U?.15 (A)
- new net RESET: U?.10 (~R), U?.10 (~R)
- new net RT: U?.4 (E)
- new net SCRL: U?.1 (B)
- new net SHIFT_4_DATA: U?.9 (QH)
- new net SHIFT_CLK: U?.11 (SCK), U?.11 (SCK)
- new net SHIFT_RCLK: U?.12 (CLK), U?.12 (CLK)
- new net UP: U?.1 (B)
- new net VCC: C?.1, C?.1, U?.16 (VCC), U?.16 (VCC)
