File: Right Main Keys.sch (KiCad schematic (older format))
At the start: 0 parts

Commit message: Schematic completed first draft
Parts:
- added C? (x3): 1n, symbol Device:C
- added U? (x3): 74LS597, symbol 74xx_IEEE:74LS597
Connections:
- new net: U?.14 (SER), U?.9 (QH) (x2)
- new net ': U?.7 (H)
- new net -: U?.5 (F)
- new net .: U?.1 (B)
- new net 0: U?.4 (E)
- new net ;: U?.6 (G)
- new net =: U?.6 (G)
- new net APP: U?.6 (G)
- new net BACK: U?.7 (H)
- new net ENTER: U?.15 (A)
- new net F10: U?.1 (B)
- new net F11: U?.2 (C)
- new net F12: U?.3 (D)
- new net F9: U?.15 (A)
- new net GND: C?.2, C?.2, C?.2, U?.13 (~SLoad), U?.13 (~SLoad), U?.13 (~SLoad), U?.14 (SER), U?.8 (GND), U?.8 (GND), U?.8 (GND)
- new net L: U?.5 (F)
- new net O: U?.15 (A)
- new net P: U?.1 (B)
- new net RALT: U?.4 (E)
- new net RCTRL: U?.7 (H)
- new net RESET: U?.10 (~R), U?.10 (~R), U?.10 (~R)
- new net RSHFT: U?.3 (D)
- new net RWIND: U?.5 (F)
- new net SHIFT_3_DATA: U?.9 (QH)
- new net SHIFT_CLK: U?.11 (SCK), U?.11 (SCK), U?.11 (SCK)
- new net SHIFT_RCLK: U?.12 (CLK), U?.12 (CLK), U?.12 (CLK)
- new net SLSH: U?.2 (C)
- new net VCC: C?.1, C?.1, C?.1, U?.16 (VCC), U?.16 (VCC), U?.16 (VCC)
- new net [: U?.2 (C)
- new net \: U?.4 (E)
- new net ]: U?.3 (D)
