File: Left Main LEDs.sch (KiCad schematic (older format))
At the start: 40 parts

Commit message: Schematic completed first draft
Parts:
- removed D?: LED F1, symbol Device:LED
- removed D?: LED F2, symbol Device:LED
- removed D?: LED F3, symbol Device:LED
- removed D?: LED `, symbol Device:LED
- removed D?: LED 1, symbol Device:LED
- removed D?: LED Q, symbol Device:LED
- removed D?: LED W, symbol Device:LED
- removed D?: LED CAPL, symbol Device:LED
- removed D?: LED S, symbol Device:LED
- removed D?: LED RSHFT, symbol Device:LED
- removed D?: LED Z, symbol Device:LED
- removed R? (x14): 1.8k, symbol Device:R
- added D?: LED F1, symbol Device:LED
- added D?: LED F2, symbol Device:LED
- added D?: LED F3, symbol Device:LED
- added D?: LED `, symbol Device:LED
- added D?: LED 1, symbol Device:LED
- added D?: LED Q, symbol Device:LED
- added D?: LED W, symbol Device:LED
- added D?: LED CAPL, symbol Device:LED
- added D?: LED S, symbol Device:LED
- added D?: LED RSHFT, symbol Device:LED
- added D?: LED Z, symbol Device:LED
- added R? (x14): 1.8k, symbol Device:R
Connections:
- net DIMMER: now also R?.2, R?.2, R?.2, R?.2, R?.2, R?.2, R?.2, R?.2, R?.2, R?.2, R?.2, R?.2, R?.2, R?.2
- net GND: now also D?.1 (K), D?.1 (K), D?.1 (K), D?.1 (K), D?.1 (K), D?.1 (K), D?.1 (K), D?.1 (K), D?.1 (K), D?.1 (K), D?.1 (K)
- net at R?.1: now also D?.2 (A) (x2)
- net at D?.2 (A): now also R?.1 (x5)
- new net: D?.2 (A), R?.1 (x9)

Commit message: Corrected errors found in design rule check
Parts:
- D100, D101, D102, D103, D104, D105, D106, D107, D108, D109, D110, D111, D112, D113, D114, D95, D96, D97, D98, D99: renamed from D?; footprint (none) -> LED_SMD:LED_1206_3216Metric_ReverseMount_Hole1.8x2.4mm
- R320, R321, R322, R323, R324, R325, R326, R327, R328, R329, R330, R331, R332, R333, R334, R335, R336, R337, R338, R339: renamed from R?; footprint (none) -> Resistor_SMD:R_1206_3216Metric_Pad1.42x1.75mm_HandSolder

Commit message: Redesigned for single large PCB
Parts:
- renumbered D95 to D55, D96 to D56, D97 to D57, D98 to D58, D99 to D59, D100 to D60, D101 to D61, D102 to D62, D103 to D63, D104 to D64, D105 to D65, D106 to D66, D107 to D67, D108 to D68, D109 to D69, D110 to D70, D111 to D71, D112 to D72, D113 to D73, D114 to D74, R320 to R200, R321 to R201, R322 to R202, R323 to R203, R324 to R204, R325 to R205, R326 to R206, R327 to R207, R328 to R208, R329 to R209, R330 to R210, R331 to R211, R332 to R212, R333 to R213, R334 to R214, R335 to R215, R336 to R216, R337 to R217, R338 to R218, R339 to R219

Commit message: PCB Routed, minor circuit changes
Parts:
- D69: value LED RSHFT -> LED LSHFT
Changed lines of the file:
@@
 $Descr B 17000 11000
 encoding utf-8
-Sheet 18 14
+Sheet 10 14
 Title ""
 Date ""
@@
 AR Path="/5E8C7194/5ECCEB56/60A6F971" Ref="D69"  Part="1"
 F 0 "D69" H 9543 6495 50  0000 C CNN
-F 1 "LED RSHFT" H 9543 6586 50  0000 C CNN
+F 1 "LED LSHFT" H 9543 6586 50  0000 C CNN
 F 2 "LED_SMD:LED_1206_3216Metric_ReverseMount_Hole1.8x2.4mm" H 9550 6750 50  0001 C CNN
 F 3 "~" H 9550 6750 50  0001 C CNN
