File: Keyboard.kicad_pcb (KiCad board)
At the start: 2 copper layers, 450.2 x 135.2 mm, 727 parts, among them J1 USB_B_Micro, J2 DEBUG, J3 USB, Q1 DMG2302U, Q2 DMG2302U, Q3 DMG2302U, SW1 SW_Push, SW10 7, SW100 ], SW101 \, SW102 L, SW103 ;, SW104 ', SW105 ENTER, SW106 ., SW107 /, SW108 RSHFT, SW109 RALT, SW11 8, SW110 RWIND, SW111 APP, SW112 RCTRL, SW12 9, SW13 E, SW14 R, SW15 T, SW16 Y, SW17 U, SW18 I, SW19 D, SW2 F4, SW20 F, SW21 G, SW22 H, SW23 J, SW24 K, SW25 C, SW26 V, SW27 B, SW28 N, SW29 M, SW3 F5, SW30 ,, SW31 SPACE, SW32 EXT1, SW33 EXT2, SW34 EXT3, SW35 EXT4, SW36 NUM LOCK, SW37 /, SW38 *, SW39 -, SW4 F6, SW40 7, SW41 8, SW42 9, SW43 +, SW44 4, SW45 5, SW46 6, SW47 1, SW48 2, SW49 3, SW5 F7, SW50 ENTER, SW51 0, SW52 ., SW53 ESC, SW54 F1, SW55 F2, SW56 F3, SW57 `, SW58 1, SW59 2, SW6 F8, SW60 3, SW61 TAB, SW62 Q, SW63 W, SW64 CAPL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

Commit message: PCB Routed, minor circuit changes
Routing:
- net GND: track 2041.3 -> 2099.2 mm, vias 9 -> 41
- net /CMK/EXT3: track 129.8 -> 127.1 mm

Commit message: Generated Manufacturing Files, small PCB details
Parts:
- added REF**: MountingHole_3.2mm_M3, MountingHole:MountingHole_3.2mm_M3, F.Cu at (52.4, 160.7)
- added REF**: MountingHole_3.2mm_M3, MountingHole:MountingHole_3.2mm_M3, F.Cu at (153.4, 35.4)
- added REF**: MountingHole_3.2mm_M3, MountingHole:MountingHole_3.2mm_M3, F.Cu at (52.4, 35.4)
- added REF**: MountingHole_3.2mm_M3, MountingHole:MountingHole_3.2mm_M3, F.Cu at (-48.7, 35.4)
- added REF**: MountingHole_3.2mm_M3, MountingHole:MountingHole_3.2mm_M3, F.Cu at (-66.7, 53.4)
- added REF**: MountingHole_3.2mm_M3, MountingHole:MountingHole_3.2mm_M3, F.Cu at (-66.7, 98.0)
- added REF**: MountingHole_3.2mm_M3, MountingHole:MountingHole_3.2mm_M3, F.Cu at (-48.8, 160.7)
- added REF**: MountingHole_3.2mm_M3, MountingHole:MountingHole_3.2mm_M3, F.Cu at (-66.7, 142.7)
- added REF**: MountingHole_3.2mm_M3, MountingHole:MountingHole_3.2mm_M3, F.Cu at (153.4, 160.7)
- added REF**: MountingHole_3.2mm_M3, MountingHole:MountingHole_3.2mm_M3, F.Cu at (254.5, 160.7)
- added REF**: MountingHole_3.2mm_M3, MountingHole:MountingHole_3.2mm_M3, F.Cu at (355.5, 160.7)
- added REF**: MountingHole_3.2mm_M3, MountingHole:MountingHole_3.2mm_M3, F.Cu at (373.5, 142.7)
- added REF**: MountingHole_3.2mm_M3, MountingHole:MountingHole_3.2mm_M3, F.Cu at (373.5, 98.0)
- added REF**: MountingHole_3.2mm_M3, MountingHole:MountingHole_3.2mm_M3, F.Cu at (373.5, 53.4)
- added REF**: MountingHole_3.2mm_M3, MountingHole:MountingHole_3.2mm_M3, F.Cu at (355.5, 35.4)
- added REF**: MountingHole_3.2mm_M3, MountingHole:MountingHole_3.2mm_M3, F.Cu at (254.5, 35.4)
Other:
- board text added: "4/26/2020"
- board text added: "Designed by lopezk38"
- board text added: "Keyboard Rev 1"
- board text added: "https://github.com/lopezk38/Custom-Keyboard"
